Commit message: changed mimic joint mechanism - now it is handled in roto-env; there is still a problme of not so accurate mimic jotin. RMS error higher that other joints; may need to do another hardware run

File: roto/assets/shadow_lite/sr_hand_touchlab.urdf (robot description, URDF)
Before this commit: robot shadowhand_motor, 26 links, 25 joints
Joints:
- joint rh_FFJ1: mimic joint=rh_FFJ2 multiplier=0 offset=0.0 -> (none)
- joint rh_MFJ1: mimic joint=rh_MFJ2 multiplier=1.0 offset=0.0 -> (none)
- joint rh_RFJ1: mimic joint=rh_RFJ2 multiplier=1.0 offset=0.0 -> (none)
